Commit message: minimalized urdf

File: spot_description/urdf/spot.urdf.xacro (robot description, xacro)
@@ -9,69 +9,5 @@
     <xacro:arg name="has_rl_kit" default="False"/>
     <xacro:arg name="has_realsense" default="False"/>
-    <xacro:arg name="kinematic_model" default="body_assist"/>
-    <xacro:property name="kinematic_model" value="$(arg kinematic_model)"/>
-    <link name="base_footprint"/>
-    <!-- Virtual Joints -->
-    <xacro:if value="${kinematic_model == 'body_assist'}">
-        <link name="body_height"/>
-        <link name="body_with_yaw"/>
-        <link name="body_with_pitch_and_yaw"/>
-        <joint name="body_height_joint" type="prismatic">
-            <parent link = "base_footprint"/>
-            <child  link = "body_height"/>
-            <axis xyz = "0 0 1"/>
-            <limit lower = "0.37" upper = "0.60" velocity="0.1" effort="1e9"/>
-        </joint>
-        <joint name="body_yaw_joint" type="revolute">
-            <parent link = "body_height"/>
-            <child  link = "body_with_yaw"/>
-            <limit lower = "${-pi/9}" upper = "${pi/9}" velocity="0.1" effort="1e9"/>
-            <axis    xyz = "0 0 1"/>
-        </joint>
-        <joint name="body_pitch_joint" type="revolute">
-            <parent link = "body_with_yaw"/>
-            <child  link = "body_with_pitch_and_yaw"/>
-            <limit lower = "${-pi/12}" upper = "${pi/12}"  velocity="0.1" effort="1e9"/>
-            <axis    xyz = "0 1 0"/>
-        </joint>
-        <joint name="body_roll_joint" type="revolute">
-            <parent link = "body_with_pitch_and_yaw"/>
-            <child  link = "body"/>
-            <limit lower = "${-pi/18}" upper = "${pi/18}"  velocity="0.1" effort="1e9"/>
-            <axis    xyz = "1 0 0"/>
-        </joint>
-    </xacro:if>
-    <xacro:if value="${kinematic_model == 'mobile_manipulation'}">
-        <!-- Virtual Base Movement links -->
-        <link name="body_x"/>
-        <link name="body_y"/>
-        <link name="body_or"/>
-        <!-- Virtual Joints -->
-        <joint name="body_x" type="prismatic">
-            <parent link = "base_footprint"/>
-            <child  link = "body_x"/>
-            <axis xyz = "1 0 0"/>
-            <limit lower = "-10.0" upper = "10.0" velocity="0.1" effort="1e9"/>
-        </joint>
-        <joint name="body_y" type="prismatic">
-            <parent link = "body_x"/>
-            <child  link = "body_y"/>
-            <axis xyz = "0 1 0"/>
-            <limit lower = "-10.0" upper = "10.0" velocity="0.1" effort="1e9"/>
-        </joint>
-        <joint name="body_or" type="revolute">
-            <parent link = "body_y"/>
-            <child  link = "body_or"/>
-            <limit lower = "0" upper = "${2*pi}" velocity="0.1" effort="1e9"/>
-            <axis    xyz = "0 0 1"/>
-        </joint>
-        <joint name="ground_to_body" type="fixed">
-            <parent link = "body_or"/>
-            <child  link = "body"/>
-            <origin xyz="0 0 0.52"/>
-        </joint>
-        <!-- EOF Virtual Base Movement Links-->
-    </xacro:if>
-    <!-- Fixed links -->
+    <link name="base_link"/>
     <link name="body">
         <visual>
@@ -86,13 +22,12 @@
         </collision>
         <inertial>
-             <mass value="16.25" />
-             <inertia  ixx="0.085" ixy="0.0"  ixz="0.0"  iyy="1.045"  iyz="0.0"  izz="1.042" />
-    	</inertial>
-    </link>
-    <link name="base_link"/>
+            <mass value="16.25" />
+            <inertia  ixx="0.085" ixy="0.0"  ixz="0.0"  iyy="1.045"  iyz="0.0"  izz="1.042" />
+        </inertial>
+    </link>
     <joint name="base_link_joint" type="fixed">
         <origin xyz="0 0 0" rpy="0 0 0" />
-        <parent link="body" />
-        <child link="base_link" />
+        <parent link="base_link" />
+        <child link="body" />
     </joint>
     <link name="front_rail"/>

Commit message: testing, still dies corrupted size vs. prev_size when using moveit from source

File: spot_description/urdf/spot.urdf.xacro (robot description, xacro)
@@ -9,5 +9,4 @@
     <xacro:arg name="has_rl_kit" default="False"/>
     <xacro:arg name="has_realsense" default="False"/>
-    <link name="base_link"/>
     <link name="body">
         <visual>
@@ -26,8 +25,9 @@
         </inertial>
     </link>
+    <link name="base_link"/>
     <joint name="base_link_joint" type="fixed">
         <origin xyz="0 0 0" rpy="0 0 0" />
-        <parent link="base_link" />
-        <child link="body" />
+        <parent link="body" />
+        <child link="base_link" />
     </joint>
     <link name="front_rail"/>
